File: MainBoard_2023/MainBoard/GNSS.kicad_sch (KiCad schematic)
At the start: 0 parts

Commit message: GNSSモジュール
Parts:
- added ANT?: SAM-M10Q-00B, SAMM10Q00B, symbol SAM-M10Q-00B:SAM-M10Q-00B
- added BT?: 6.8MM_COIN_CELL, SparkFun_Ublox SAM-M8Q:ML414H_IV01E, symbol SparkFun_Ublox SAM-M8Q-eagle-import:ML414H_IV01E_BATTERY
- added C? (x2): 1.0uF, symbol Device:C_Small
- added D?: Yellow, SparkFun_Ublox SAM-M8Q:LED-0603, symbol SparkFun_Ublox SAM-M8Q-eagle-import:LED-YELLOW0603
- added D?: 0.5A/40V/420mV, SparkFun_Ublox SAM-M8Q:SOD-323, symbol SparkFun_Ublox SAM-M8Q-eagle-import:DIODE-SCHOTTKY-PMEG4005EJ
- added J?: CONN_08NO_SILK_FEMALE_PTH, SparkFun_Ublox SAM-M8Q:1X08_NO_SILK, symbol SparkFun_Ublox SAM-M8Q-eagle-import:CONN_08NO_SILK_FEMALE_PTH
- added J?: BOOT, SparkFun_Ublox SAM-M8Q:1X06_NO_SILK, symbol SparkFun_Ublox SAM-M8Q-eagle-import:CONN_06NO_SILK_NO_POP
- added JP?: SolderJumper_3_Bridged123, symbol Jumper:SolderJumper_3_Bridged123
- added JP?: SolderJumper_2_Bridged, symbol Jumper:SolderJumper_2_Bridged
- added R? (x2): 470, symbol Device:R_Small
- added R? (x2): 22, symbol Device:R_Small
- added R?: 1k, SparkFun_Ublox SAM-M8Q:0603, symbol SparkFun_Ublox SAM-M8Q-eagle-import:1KOHM-0603-1/10W-1%
- added R? (x2): 2.2k, symbol Device:R_Small
- added R?: 3.3k, SparkFun_Ublox SAM-M8Q:0603, symbol SparkFun_Ublox SAM-M8Q-eagle-import:3.3KOHM-0603-1/10W-1%
Connections:
- new net: ANT?.14 (RXD), R?.1
- new net: ANT?.12 (SCL), R?.1
- new net: D?.A, R?.1
- new net: JP?.1 (A), R?.2 (x2)
- new net: ANT?.13 (TXD), R?.1
- new net: JP?.3 (B), R?.2
- new net: ANT?.9 (SDA), R?.1
- new net: D?.C, R?.2
- new net +3.3V: ANT?.17 (VCC), ANT?.2 (V_IO), C?.1, D?.A, J?.3, J?.3, JP?.2 (C)
- new net BACKUP: ANT?.3 (V_BCKP), BT?.+, C?.1, R?.1
- new net GND: ANT?.1 (GND_1), ANT?.10 (GND_5), ANT?.11 (GND_6), ANT?.15 (GND_7), ANT?.16 (GND_8), ANT?.20 (GND_9), ANT?.4 (GND_2), ANT?.5 (GND_3), ANT?.6 (GND_4), BT?.-, C?.2, C?.2, D?.C, J?.1, J?.2, J?.4
- new net INT: ANT?.19 (EXTINT), J?.5
- new net PPS: ANT?.7 (TIMEPULSE), J?.8, JP?.2 (B)
- new net RXI: J?.4, R?.2
- new net SCL: J?.1, R?.1, R?.2
- new net SDA: J?.2, R?.1, R?.2
- new net TXO: J?.5, R?.2
- new net ~{RESET}: ANT?.18 (RESET_N), J?.7
- new net ~{SAFE}: ANT?.8 (SAFEBOOT_N), J?.6
Other:
- note added: "7-bit unshifted I2C address: 0x10"
- note added: "Battery Initial Charge: 2.3-2.8V Battery Charge Rate: 1mA MAX Voff: 2.0V 72 hours charge time from 2.0-3.1V"
- note added: "Connectors"
- note added: "Cut Jumper to disable PPS LED"
- note added: "Cut Jumper to remove I2C pullups from bus"
- note added: "Pulse Per Second LED"
- note added: "RTC Backup"
- note added: "Ublox SAM-M8Q"

Commit message: メイン基板設計一段落
Parts:
- removed BT?: 6.8MM_COIN_CELL, SparkFun_Ublox SAM-M8Q:ML414H_IV01E, symbol SparkFun_Ublox SAM-M8Q-eagle-import:ML414H_IV01E_BATTERY
- removed D?: Yellow, SparkFun_Ublox SAM-M8Q:LED-0603, symbol SparkFun_Ublox SAM-M8Q-eagle-import:LED-YELLOW0603
- removed D?: 0.5A/40V/420mV, SparkFun_Ublox SAM-M8Q:SOD-323, symbol SparkFun_Ublox SAM-M8Q-eagle-import:DIODE-SCHOTTKY-PMEG4005EJ
- removed J?: CONN_08NO_SILK_FEMALE_PTH, SparkFun_Ublox SAM-M8Q:1X08_NO_SILK, symbol SparkFun_Ublox SAM-M8Q-eagle-import:CONN_08NO_SILK_FEMALE_PTH
- removed J?: BOOT, SparkFun_Ublox SAM-M8Q:1X06_NO_SILK, symbol SparkFun_Ublox SAM-M8Q-eagle-import:CONN_06NO_SILK_NO_POP
- removed R?: 1k, SparkFun_Ublox SAM-M8Q:0603, symbol SparkFun_Ublox SAM-M8Q-eagle-import:1KOHM-0603-1/10W-1%
- removed R?: 3.3k, SparkFun_Ublox SAM-M8Q:0603, symbol SparkFun_Ublox SAM-M8Q-eagle-import:3.3KOHM-0603-1/10W-1%
- added BT?: ML-1220_F1AN, ML-1220F1AN, symbol ML-1220_F1AN:ML-1220_F1AN
- added D?: CUHS20S30,H3F, CUHS20S40H3F, symbol CUHS20S30:CUHS20S30,H3F
- added D?: LED_Small, symbol Device:LED_Small
- added R?: 1.4k, symbol Device:R_Small
- added R?: 1k, symbol Device:R_Small
- JP?: value SolderJumper_3_Bridged123 -> SolderJumper
- JP?: value SolderJumper_2_Bridged -> SolderJumper
Connections:
- net +3.3V: now also D?.2
- net BACKUP: now also BT?.1 (+), R?.2
- net GND: now also BT?.2 (-), D?.1 (K)
- net at JP?.1 (A): now also R?.1
- net RXI renamed RX
- net TXO renamed TX
- net ~{RESET} renamed RESET
- net ~{SAFE} renamed SAFE
- new net: D?.1, R?.1
- new net: D?.2 (A), R?.2
Other:
- note added: "Battery Initial Charge: 3.0-3.3V Battery Charge Rate: 1mA MAX Voff: 2.0V"
- note added: "Cut Jumper to disable Pulse Per Second LED"
- note added: "Ublox SAM-M10Q"
- note removed: "Battery Initial Charge: 2.3-2.8V Battery Charge Rate: 1mA MAX Voff: 2.0V 72 hours charge time from 2.0-3.1V"
- note removed: "Connectors"
- note removed: "Cut Jumper to disable PPS LED"
- note removed: "Pulse Per Second LED"
- note removed: "Ublox SAM-M8Q"
- moved on the sheet: ANT?, C?, JP?, R?

Commit message: ERC通った
Parts:
- gave numbers to parts that had none: 16
Changed lines of the file:
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@@
   (symbol (lib_id "Device:R_Small") (at 180.34 96.52 90) (unit 1)
     (in_bom yes) (on_board yes)
-    (property "Reference" "R?" (id 0) (at 176.53 97.79 90))
+    (property "Reference" "R47" (id 0) (at 176.53 97.79 90))
     (property "Value" "470" (id 1) (at 180.34 96.52 90))
     (property "Footprint" "" (id 2) (at 180.34 96.52 0)
@@
   (symbol (lib_id "power:+3.3V") (at 195.58 67.31 0) (unit 1)
     (in_bom yes) (on_board yes)
-    (property "Reference" "#PWR?" (id 0) (at 195.58 71.12 0)
+    (property "Reference" "#PWR0110" (id 0) (at 195.58 71.12 0)
       (effects (font (size 1.27 1.27)) hide)
     )
@@
   (symbol (lib_id "Device:R_Small") (at 180.34 88.9 90) (unit 1)
     (in_bom yes) (on_board yes)
-    (property "Reference" "R?" (id 0) (at 176.53 90.17 90))
+    (property "Reference" "R45" (id 0) (at 176.53 90.17 90))
     (property "Value" "22" (id 1) (at 180.34 88.9 90))
     (property "Footprint" "" (id 2) (at 180.34 88.9 0)
@@
   (symbol (lib_id "CUHS20S30:CUHS20S30,H3F") (at 87.63 72.39 90) (unit 1)
     (in_bom yes) (on_board yes)
-    (property "Reference" "D?" (id 0) (at 81.28 67.31 90)
+    (property "Reference" "D1" (id 0) (at 81.28 67.31 90)
       (effects (font (size 1.27 1.27)) (justify right))
     )
@@
   (symbol (lib_id "power:+3.3V") (at 135.89 96.52 0) (unit 1)
     (in_bom yes) (on_board yes)
-    (property "Reference" "#PWR?" (id 0) (at 135.89 100.33 0)
+    (property "Reference" "#PWR0105" (id 0) (at 135.89 100.33 0)
       (effects (font (size 1.27 1.27)) hide)
     )
@@
   (symbol (lib_id "Device:R_Small") (at 180.34 93.98 90) (unit 1)
     (in_bom yes) (on_board yes)
-    (property "Reference" "R?" (id 0) (at 176.53 92.71 90))
+    (property "Reference" "R46" (id 0) (at 176.53 92.71 90))
     (property "Value" "470" (id 1) (at 180.34 93.98 90))
     (property "Footprint" "" (id 2) (at 180.34 93.98 0)
@@
   (symbol (lib_id "Jumper:SolderJumper_3_Bridged123") (at 195.58 73.66 180) (unit 1)
     (in_bom yes) (on_board yes)
-    (property "Reference" "JP?" (id 0) (at 199.39 69.85 0))
+    (property "Reference" "JP4" (id 0) (at 199.39 69.85 0))
     (property "Value" "SolderJumper" (id 1) (at 204.47 72.39 0))
     (property "Footprint" "" (id 2) (at 195.58 73.66 0)
@@
   (symbol (lib_id "Device:R_Small") (at 200.66 80.01 180) (unit 1)
     (in_bom yes) (on_board yes)
-    (property "Reference" "R?" (id 0) (at 204.47 78.74 0))
+    (property "Reference" "R49" (id 0) (at 204.47 78.74 0))
     (property "Value" "2.2k" (id 1) (at 204.47 81.28 0))
     (property "Footprint" "" (id 2) (at 200.66 80.01 0)
@@
   (symbol (lib_id "power:GND") (at 135.89 106.68 0) (unit 1)
     (in_bom yes) (on_board yes)
-    (property "Reference" "#PWR?" (id 0) (at 135.89 113.03 0)
+    (property "Reference" "#PWR0106" (id 0) (at 135.89 113.03 0)
       (effects (font (size 1.27 1.27)) hide)
     )
@@
   (symbol (lib_id "Device:C_Small") (at 135.89 101.6 0) (unit 1)
     (in_bom yes) (on_board yes) (fields_autoplaced)
-    (property "Reference" "C?" (id 0) (at 138.2141 100.7716 0)
+    (property "Reference" "C25" (id 0) (at 138.2141 100.7716 0)
       (effects (font (size 1.27 1.27)) (justify left))
     )
@@
   (symbol (lib_id "Device:C_Small") (at 102.87 85.09 0) (unit 1)
     (in_bom yes) (on_board yes) (fields_autoplaced)
-    (property "Reference" "C?" (id 0) (at 105.1941 84.2616 0)
+    (property "Reference" "C24" (id 0) (at 105.1941 84.2616 0)
       (effects (font (size 1.27 1.27)) (justify left))
     )
@@
   (symbol (lib_id "power:+3.3V") (at 146.05 76.2 0) (unit 1)
     (in_bom yes) (on_board yes)
-    (property "Reference" "#PWR?" (id 0) (at 146.05 80.01 0)
+    (property "Reference" "#PWR0107" (id 0) (at 146.05 80.01 0)
       (effects (font (size 1.27 1.27)) hide)
     )
@@
   (symbol (lib_id "power:GND") (at 177.8 121.92 0) (unit 1)
     (in_bom yes) (on_board yes)
-    (property "Reference" "#PWR?" (id 0) (at 177.8 128.27 0)
+    (property "Reference" "#PWR0109" (id 0) (at 177.8 128.27 0)
       (effects (font (size 1.27 1.27)) hide)
     )
@@
   (symbol (lib_id "Device:R_Small") (at 87.63 74.93 0) (unit 1)
     (in_bom yes) (on_board yes) (fields_autoplaced)
-    (property "Reference" "R?" (id 0) (at 89.1286 74.0953 0)
+    (property "Reference" "R42" (id 0) (at 89.1286 74.0953 0)
       (effects (font (size 1.27 1.27)) (justify left))
     )
@@
   (symbol (lib_id "power:GND") (at 87.63 90.17 0) (unit 1)
     (in_bom yes) (on_board yes)
-    (property "Reference" "#PWR?" (id 0) (at 87.63 96.52 0)
+    (property "Reference" "#PWR0103" (id 0) (at 87.63 96.52 0)
       (effects (font (size 1.27 1.27)) hide)
     )
@@
   (symbol (lib_id "power:GND") (at 146.05 106.68 0) (unit 1)
     (in_bom yes) (on_board yes)
-    (property "Reference" "#PWR?" (id 0) (at 146.05 113.03 0)
+    (property "Reference" "#PWR0108" (id 0) (at 146.05 113.03 0)
       (effects (font (size 1.27 1.27)) hide)
     )
@@
   (symbol (lib_id "Device:R_Small") (at 177.8 114.3 0) (unit 1)
     (in_bom yes) (on_board yes) (fields_autoplaced)
-    (property "Reference" "R?" (id 0) (at 179.2986 113.4653 0)
+    (property "Reference" "R43" (id 0) (at 179.2986 113.4653 0)
       (effects (font (size 1.27 1.27)) (justify left))
     )
@@
   (symbol (lib_id "ML-1220_F1AN:ML-1220_F1AN") (at 87.63 83.82 0) (mirror y) (unit 1)
     (in_bom yes) (on_board yes) (fields_autoplaced)
-    (property "Reference" "BT?" (id 0) (at 77.47 77.631 0))
+    (property "Reference" "BT1" (id 0) (at 77.47 77.631 0))
     (property "Value" "ML-1220_F1AN" (id 1) (at 77.47 80.1679 0))
     (property "Footprint" "ML-1220F1AN" (id 2) (at 71.12 81.28 0)
@@
   (symbol (lib_id "SAM-M10Q-00B:SAM-M10Q-00B") (at 160.02 91.44 0) (unit 1)
     (in_bom yes) (on_board yes) (fields_autoplaced)
-    (property "Reference" "ANT?" (id 0) (at 160.02 72.551 0))
+    (property "Reference" "ANT1" (id 0) (at 160.02 72.551 0))
     (property "Value" "SAM-M10Q-00B" (id 1) (at 160.02 75.0879 0))
     (property "Footprint" "SAMM10Q00B" (id 2) (at 177.8 92.71 0)
@@
   (symbol (lib_id "Device:R_Small") (at 180.34 86.36 90) (unit 1)
     (in_bom yes) (on_board yes)
-    (property "Reference" "R?" (id 0) (at 176.53 85.09 90))
+    (property "Reference" "R44" (id 0) (at 176.53 85.09 90))
     (property "Value" "22" (id 1) (at 180.34 86.36 90))
     (property "Footprint" "" (id 2) (at 180.34 86.36 0)
@@
   (symbol (lib_id "Jumper:SolderJumper_2_Bridged") (at 177.8 107.95 90) (unit 1)
     (in_bom yes) (on_board yes)
-    (property "Reference" "JP?" (id 0) (at 175.26 106.68 90))
+    (property "Reference" "JP3" (id 0) (at 175.26 106.68 90))
     (property "Value" "SolderJumper" (id 1) (at 170.18 109.22 90))
     (property "Footprint" "" (id 2) (at 177.8 107.95 0)
@@
   (symbol (lib_id "Device:R_Small") (at 190.5 80.01 180) (unit 1)
     (in_bom yes) (on_board yes)
-    (property "Reference" "R?" (id 0) (at 194.31 78.74 0))
+    (property "Reference" "R48" (id 0) (at 194.31 78.74 0))
     (property "Value" "2.2k" (id 1) (at 194.31 81.28 0))
     (property "Footprint" "" (id 2) (at 190.5 80.01 0)
@@
   (symbol (lib_id "power:GND") (at 102.87 90.17 0) (unit 1)
     (in_bom yes) (on_board yes)
-    (property "Reference" "#PWR?" (id 0) (at 102.87 96.52 0)
+    (property "Reference" "#PWR0104" (id 0) (at 102.87 96.52 0)
       (effects (font (size 1.27 1.27)) hide)
     )
@@
   (symbol (lib_id "power:+3.3V") (at 87.63 63.5 0) (unit 1)
     (in_bom yes) (on_board yes)
-    (property "Reference" "#PWR?" (id 0) (at 87.63 67.31 0)
+    (property "Reference" "#PWR0102" (id 0) (at 87.63 67.31 0)
       (effects (font (size 1.27 1.27)) hide)
     )
@@
   (symbol (lib_id "Device:LED_Small") (at 177.8 119.38 90) (unit 1)
     (in_bom yes) (on_board yes) (fields_autoplaced)
-    (property "Reference" "D?" (id 0) (at 179.578 118.4818 90)
+    (property "Reference" "D2" (id 0) (at 179.578 118.4818 90)
       (effects (font (size 1.27 1.27)) (justify right))
     )

Commit message: フットプリントをすべて割り当て
Parts:
- ANT1: footprint SAMM10Q00B -> SAM-M10Q-00B:SAM-M10Q-00B
- BT1: footprint ML-1220F1AN -> ML-1220_F1AN:ML-1220_F1AN
- C24, C25: footprint (none) -> Capacitor_SMD:C_0603_1608Metric_Pad1.08x0.95mm_HandSolder
- D1: footprint CUHS20S40H3F -> CUHS20S30:CUHS20S30
- D2: footprint (none) -> LED_SMD:LED_1206_3216Metric_Pad1.42x1.75mm_HandSolder
- JP3: footprint (none) -> Jumper:SolderJumper-2_P1.3mm_Open_TrianglePad1.0x1.5mm
- JP4: footprint (none) -> Jumper:SolderJumper-3_P2.0mm_Open_TrianglePad1.0x1.5mm_NumberLabels
- R42, R43, R44, R45, R46, R47, R48, R49: footprint (none) -> Resistor_SMD:R_0603_1608Metric_Pad0.98x0.95mm_HandSolder
Changed lines of the file:
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@@
     (property "Reference" "R47" (id 0) (at 176.53 97.79 90))
     (property "Value" "470" (id 1) (at 180.34 96.52 90))
-    (property "Footprint" "" (id 2) (at 180.34 96.52 0)
+    (property "Footprint" "Resistor_SMD:R_0603_1608Metric_Pad0.98x0.95mm_HandSolder" (id 2) (at 180.34 96.52 0)
       (effects (font (size 1.27 1.27)) hide)
     )
@@
   (symbol (lib_id "power:+3.3V") (at 195.58 67.31 0) (unit 1)
     (in_bom yes) (on_board yes)
-    (property "Reference" "#PWR0110" (id 0) (at 195.58 71.12 0)
+    (property "Reference" "#PWR0111" (id 0) (at 195.58 71.12 0)
       (effects (font (size 1.27 1.27)) hide)
     )
@@
     (property "Reference" "R45" (id 0) (at 176.53 90.17 90))
     (property "Value" "22" (id 1) (at 180.34 88.9 90))
-    (property "Footprint" "" (id 2) (at 180.34 88.9 0)
+    (property "Footprint" "Resistor_SMD:R_0603_1608Metric_Pad0.98x0.95mm_HandSolder" (id 2) (at 180.34 88.9 0)
       (effects (font (size 1.27 1.27)) hide)
     )
@@
       (effects (font (size 1.27 1.27)) (justify right))
     )
-    (property "Footprint" "CUHS20S40H3F" (id 2) (at 83.82 64.77 0)
+    (property "Footprint" "CUHS20S30:CUHS20S30" (id 2) (at 83.82 64.77 0)
       (effects (font (size 1.27 1.27)) (justify left) hide)
     )
@@
   (symbol (lib_id "power:+3.3V") (at 135.89 96.52 0) (unit 1)
     (in_bom yes) (on_board yes)
-    (property "Reference" "#PWR0105" (id 0) (at 135.89 100.33 0)
+    (property "Reference" "#PWR0106" (id 0) (at 135.89 100.33 0)
       (effects (font (size 1.27 1.27)) hide)
     )
@@
     (property "Reference" "R46" (id 0) (at 176.53 92.71 90))
     (property "Value" "470" (id 1) (at 180.34 93.98 90))
-    (property "Footprint" "" (id 2) (at 180.34 93.98 0)
+    (property "Footprint" "Resistor_SMD:R_0603_1608Metric_Pad0.98x0.95mm_HandSolder" (id 2) (at 180.34 93.98 0)
       (effects (font (size 1.27 1.27)) hide)
     )
@@
     (property "Reference" "JP4" (id 0) (at 199.39 69.85 0))
     (property "Value" "SolderJumper" (id 1) (at 204.47 72.39 0))
-    (property "Footprint" "" (id 2) (at 195.58 73.66 0)
+    (property "Footprint" "Jumper:SolderJumper-3_P2.0mm_Open_TrianglePad1.0x1.5mm_NumberLabels" (id 2) (at 195.58 73.66 0)
       (effects (font (size 1.27 1.27)) hide)
     )
@@
     (property "Reference" "R49" (id 0) (at 204.47 78.74 0))
     (property "Value" "2.2k" (id 1) (at 204.47 81.28 0))
-    (property "Footprint" "" (id 2) (at 200.66 80.01 0)
+    (property "Footprint" "Resistor_SMD:R_0603_1608Metric_Pad0.98x0.95mm_HandSolder" (id 2) (at 200.66 80.01 0)
       (effects (font (size 1.27 1.27)) hide)
     )
@@
   (symbol (lib_id "power:GND") (at 135.89 106.68 0) (unit 1)
     (in_bom yes) (on_board yes)
-    (property "Reference" "#PWR0106" (id 0) (at 135.89 113.03 0)
+    (property "Reference" "#PWR0107" (id 0) (at 135.89 113.03 0)
       (effects (font (size 1.27 1.27)) hide)
     )
@@
       (effects (font (size 1.27 1.27)) (justify left))
     )
-    (property "Footprint" "" (id 2) (at 135.89 101.6 0)
+    (property "Footprint" "Capacitor_SMD:C_0603_1608Metric_Pad1.08x0.95mm_HandSolder" (id 2) (at 135.89 101.6 0)
       (effects (font (size 1.27 1.27)) hide)
     )
@@
       (effects (font (size 1.27 1.27)) (justify left))
     )
-    (property "Footprint" "" (id 2) (at 102.87 85.09 0)
+    (property "Footprint" "Capacitor_SMD:C_0603_1608Metric_Pad1.08x0.95mm_HandSolder" (id 2) (at 102.87 85.09 0)
       (effects (font (size 1.27 1.27)) hide)
     )
@@
   (symbol (lib_id "power:+3.3V") (at 146.05 76.2 0) (unit 1)
     (in_bom yes) (on_board yes)
-    (property "Reference" "#PWR0107" (id 0) (at 146.05 80.01 0)
+    (property "Reference" "#PWR0108" (id 0) (at 146.05 80.01 0)
       (effects (font (size 1.27 1.27)) hide)
     )
@@
   (symbol (lib_id "power:GND") (at 177.8 121.92 0) (unit 1)
     (in_bom yes) (on_board yes)
-    (property "Reference" "#PWR0109" (id 0) (at 177.8 128.27 0)
+    (property "Reference" "#PWR0110" (id 0) (at 177.8 128.27 0)
       (effects (font (size 1.27 1.27)) hide)
     )
@@
       (effects (font (size 1.27 1.27)) (justify left))
     )
-    (property "Footprint" "" (id 2) (at 87.63 74.93 0)
+    (property "Footprint" "Resistor_SMD:R_0603_1608Metric_Pad0.98x0.95mm_HandSolder" (id 2) (at 87.63 74.93 0)
       (effects (font (size 1.27 1.27)) hide)
     )
@@
   (symbol (lib_id "power:GND") (at 87.63 90.17 0) (unit 1)
     (in_bom yes) (on_board yes)
-    (property "Reference" "#PWR0103" (id 0) (at 87.63 96.52 0)
+    (property "Reference" "#PWR0104" (id 0) (at 87.63 96.52 0)
       (effects (font (size 1.27 1.27)) hide)
     )
@@
   (symbol (lib_id "power:GND") (at 146.05 106.68 0) (unit 1)
     (in_bom yes) (on_board yes)
-    (property "Reference" "#PWR0108" (id 0) (at 146.05 113.03 0)
+    (property "Reference" "#PWR0109" (id 0) (at 146.05 113.03 0)
       (effects (font (size 1.27 1.27)) hide)
     )
@@
       (effects (font (size 1.27 1.27)) (justify left))
     )
-    (property "Footprint" "" (id 2) (at 177.8 114.3 0)
+    (property "Footprint" "Resistor_SMD:R_0603_1608Metric_Pad0.98x0.95mm_HandSolder" (id 2) (at 177.8 114.3 0)
       (effects (font (size 1.27 1.27)) hide)
     )
@@
     (property "Reference" "BT1" (id 0) (at 77.47 77.631 0))
     (property "Value" "ML-1220_F1AN" (id 1) (at 77.47 80.1679 0))
-    (property "Footprint" "ML-1220F1AN" (id 2) (at 71.12 81.28 0)
+    (property "Footprint" "ML-1220_F1AN:ML-1220_F1AN" (id 2) (at 71.12 81.28 0)
       (effects (font (size 1.27 1.27)) (justify left) hide)
     )
@@
     (property "Reference" "ANT1" (id 0) (at 160.02 72.551 0))
     (property "Value" "SAM-M10Q-00B" (id 1) (at 160.02 75.0879 0))
-    (property "Footprint" "SAMM10Q00B" (id 2) (at 177.8 92.71 0)
+    (property "Footprint" "SAM-M10Q-00B:SAM-M10Q-00B" (id 2) (at 177.8 92.71 0)
       (effects (font (size 1.27 1.27)) (justify left) hide)
     )
@@
     (property "Reference" "R44" (id 0) (at 176.53 85.09 90))
     (property "Value" "22" (id 1) (at 180.34 86.36 90))
-    (property "Footprint" "" (id 2) (at 180.34 86.36 0)
+    (property "Footprint" "Resistor_SMD:R_0603_1608Metric_Pad0.98x0.95mm_HandSolder" (id 2) (at 180.34 86.36 0)
       (effects (font (size 1.27 1.27)) hide)
     )
@@
     (property "Reference" "JP3" (id 0) (at 175.26 106.68 90))
     (property "Value" "SolderJumper" (id 1) (at 170.18 109.22 90))
-    (property "Footprint" "" (id 2) (at 177.8 107.95 0)
+    (property "Footprint" "Jumper:SolderJumper-2_P1.3mm_Open_TrianglePad1.0x1.5mm" (id 2) (at 177.8 107.95 0)
       (effects (font (size 1.27 1.27)) hide)
     )
@@
     (property "Reference" "R48" (id 0) (at 194.31 78.74 0))
     (property "Value" "2.2k" (id 1) (at 194.31 81.28 0))
-    (property "Footprint" "" (id 2) (at 190.5 80.01 0)
+    (property "Footprint" "Resistor_SMD:R_0603_1608Metric_Pad0.98x0.95mm_HandSolder" (id 2) (at 190.5 80.01 0)
       (effects (font (size 1.27 1.27)) hide)
     )
@@
   (symbol (lib_id "power:GND") (at 102.87 90.17 0) (unit 1)
     (in_bom yes) (on_board yes)
-    (property "Reference" "#PWR0104" (id 0) (at 102.87 96.52 0)
+    (property "Reference" "#PWR0105" (id 0) (at 102.87 96.52 0)
       (effects (font (size 1.27 1.27)) hide)
     )
@@
   (symbol (lib_id "power:+3.3V") (at 87.63 63.5 0) (unit 1)
     (in_bom yes) (on_board yes)
-    (property "Reference" "#PWR0102" (id 0) (at 87.63 67.31 0)
+    (property "Reference" "#PWR0103" (id 0) (at 87.63 67.31 0)
       (effects (font (size 1.27 1.27)) hide)
     )
@@
       (effects (font (size 1.27 1.27)) (justify right))
     )
-    (property "Footprint" "" (id 2) (at 177.8 119.38 90)
-      (effects (font (size 1.27 1.27)) hide)
-    )
+    (property "Footprint" "LED_SMD:LED_1206_3216Metric_Pad1.42x1.75mm_HandSolder" (id 2) (at 177.8 119.38 90)
+      (effects (font (size 1.27 1.27)) hide)
+    )
