File: MainBoard_2023/MainBoard_rev2/MainBoard.kicad_sch (KiCad schematic)
At the start: 49 parts, among them J1 Conn_01x02, J2 USB1125-GF-B_REVA, J3 Conn_01x03, J4 Conn_01x03, J5 Micro_SD_Card_Det_Hirose_DM3AT, J6 Micro_SD_Card_Det_Hirose_DM3AT, U1 BNO055, U2 ICP-10111, U3 Pi Pico 0, U4 XIAO, U5 Pi Pico 1

Commit message: 配線終了
Parts:
- removed S2: B3AL, B3AL-1002P-MS:B3AL-1002P-MS, symbol B3AL-1002P-MS:B3AL-1002P-MS
Connections:
- net SW1: no longer names the net of U3.26 (GP20)
- no-connect marks 50 -> 51
Changed lines of the file:
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@@
   (junction (at 214.63 92.71) (diameter 0) (color 0 0 0 0)
   )
-  (junction (at 52.07 38.1) (diameter 0) (color 0 0 0 0)
-  )
   (junction (at 25.4 172.72) (diameter 0) (color 0 0 0 0)
   )
@@
   (no_connect (at 175.26 38.1))
   (no_connect (at 175.26 40.64))
+  (no_connect (at 96.52 63.5))
   (no_connect (at 148.59 66.04))
   (no_connect (at 175.26 68.58))
@@
     (stroke (width 0) (type default) (color 0 0 0 0))
   )
-  (wire (pts (xy 59.69 27.94) (xy 60.96 27.94))
-    (stroke (width 0) (type default) (color 0 0 0 0))
-  )
   (wire (pts (xy 220.98 127) (xy 224.79 127))
     (stroke (width 0) (type default) (color 0 0 0 0))
@@
     (stroke (width 0) (type default) (color 0 0 0 0))
   )
-  (wire (pts (xy 52.07 27.94) (xy 57.15 27.94))
-    (stroke (width 0) (type default) (color 0 0 0 0))
-  )
   (wire (pts (xy 280.67 127) (xy 280.67 120.65))
     (stroke (width 0) (type default) (color 0 0 0 0))
@@
     (stroke (width 0) (type default) (color 0 0 0 0))
   )
-  (wire (pts (xy 52.07 27.94) (xy 52.07 38.1))
-    (stroke (width 0) (type default) (color 0 0 0 0))
-  )
   (wire (pts (xy 33.02 26.67) (xy 35.56 26.67))
     (stroke (width 0) (type default) (color 0 0 0 0))
@@
     (effects (font (size 1.27 1.27)) (justify right bottom))
   )
-  (label "SW1" (at 96.52 63.5 180)
-    (effects (font (size 1.27 1.27)) (justify right bottom))
-  )
   (label "SDA0" (at 40.64 102.87 0)
     (effects (font (size 1.27 1.27)) (justify left bottom))
@@
     (effects (font (size 1.27 1.27)) (justify left bottom))
   )
-  (label "SW1" (at 60.96 27.94 0)
-    (effects (font (size 1.27 1.27)) (justify left bottom))
-  )
   (label "SW3" (at 96.52 68.58 180)
     (effects (font (size 1.27 1.27)) (justify right bottom))
@@
     (pin "2")
   )
-  (symbol (lib_id "B3AL-1002P-MS:B3AL-1002P-MS") (at 59.69 27.94 270) (mirror x) (unit 1)
-    (in_bom yes) (on_board yes)
-    (property "Reference" "S2" (id 0) (at 54.61 20.32 90)
-      (effects (font (size 1.27 1.27)) (justify left))
-    )
-    (property "Value" "B3AL" (id 1) (at 57.15 20.32 90)
-      (effects (font (size 1.27 1.27)) (justify left))
-    )
-    (property "Footprint" "B3AL-1002P-MS:B3AL-1002P-MS" (id 2) (at 55.88 20.32 0)
-      (effects (font (size 1.27 1.27)) (justify left) hide)
-    )
-    (property "Datasheet" "https://componentsearchengine.com/Datasheets/1/B3AL-1002P-MS.pdf" (id 3) (at 53.34 20.32 0)
-      (effects (font (size 1.27 1.27)) (justify left) hide)
-    )
-    (property "Description" "OMRON ELECTRONIC COMPONENTS - B3AL-1002P-MS - TACTILE SWITCH, SPST-NO, 0.05A, 16V, SMT" (id 4) (at 50.8 20.32 0)
-      (effects (font (size 1.27 1.27)) (justify left) hide)
-    )
-    (property "Height" "5.4" (id 5) (at 48.26 20.32 0)
-      (effects (font (size 1.27 1.27)) (justify left) hide)
-    )
-    (property "Manufacturer_Name" "Omron Electronics" (id 6) (at 45.72 20.32 0)
-      (effects (font (size 1.27 1.27)) (justify left) hide)
-    )
-    (property "Manufacturer_Part_Number" "B3AL-1002P-MS" (id 7) (at 43.18 20.32 0)
-      (effects (font (size 1.27 1.27)) (justify left) hide)
-    )
-    (property "Mouser Part Number" "653-B3AL-1002P-MS" (id 8) (at 40.64 20.32 0)
-      (effects (font (size 1.27 1.27)) (justify left) hide)
-    )
-    (property "Mouser Price/Stock" "https://www.mouser.co.uk/ProductDetail/Omron-Electronics/B3AL-1002P-MS?qs=HXFqYaX1Q2yMcMO0j50f3A%3D%3D" (id 9) (at 38.1 20.32 0)
-      (effects (font (size 1.27 1.27)) (justify left) hide)
-    )
-    (property "Arrow Part Number" "B3AL-1002P-MS" (id 10) (at 35.56 20.32 0)
-      (effects (font (size 1.27 1.27)) (justify left) hide)
-    )
-    (property "Arrow Price/Stock" "https://www.arrow.com/en/products/b3al-1002p-ms/omron?region=nac" (id 11) (at 33.02 20.32 0)
-      (effects (font (size 1.27 1.27)) (justify left) hide)
-    )
-    (property "Mouser Testing Part Number" "" (id 12) (at 30.48 20.32 0)
-      (effects (font (size 1.27 1.27)) (justify left) hide)
-    )
-    (property "Mouser Testing Price/Stock" "" (id 13) (at 27.94 20.32 0)
-      (effects (font (size 1.27 1.27)) (justify left) hide)
-    )
-    (pin "1")
-    (pin "2")
-  )
   (symbol (lib_id "power:+3.3V") (at 44.45 95.25 270) (unit 1)
     (in_bom yes) (on_board yes)
@@
       (reference "S1") (unit 1) (value "POWER") (footprint "RS_PRO_PCB_Slide_Switch_SPDT_Latching_3A_120V_ac_Top:RS_PRO_PCB_Slide_Switch_SPDT_Latching_3A_120V_ac_Top")
     )
-    (path "/aa422979-3a6d-46ba-8f8a-073665f9f40c"
-      (reference "S2") (unit 1) (value "B3AL") (footprint "B3AL-1002P-MS:B3AL-1002P-MS")
-    )
     (path "/466d18fc-a229-4d5a-a523-a2c4f33aefd7"
