File: CyclingPowerMeter_2023/MainBoard/MainBoard.kicad_sch (KiCad schematic)
At the start: 34 parts, among them J1 Conn_01x01, J10 S2B-PH-SM4-TB_LF__SN_, J11 Conn_01x01, J12 Conn_01x01, J2 Conn_01x01, J3 Conn_01x01, J4 Conn_01x01, J5 Conn_01x01, J6 Conn_01x01, J7 Conn_01x01, J8 Conn_01x01, J9 BLA05-05S30, SW1 RS_PRO_PCB_Slide_Switch_SPDT_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, U1 ADS122U04IPW, U2 Seeed_Studio_XIAO_nRF52840_Se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

Commit message: PMのファームウェアを編集中
Parts:
- C5, C7: value C_Small -> 0.01u
- C6: value C_Small -> 0.1u
- R1, R2: value R_Small -> 5.1k
Other:
- note added: "1"
- note added: "2"
- note added: "3"
- note added: "4"
- note added: "CutOff=149Hz"
- note added: "minus"
- note added: "plus"
- note added: "↓"
- note added: "クランク"
- note added: "力"
- note added: "増える"
- note added: "減る"
- note added: "軸"
Changed lines of the file:
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@@
     (stroke (width 0) (type default) (color 0 0 0 0))
+  )
+  (polyline (pts (xy 48.26 109.22) (xy 46.99 109.22))
+    (stroke (width 0) (type solid) (color 0 0 0 0))
   )
   (wire (pts (xy 92.71 55.88) (xy 99.06 55.88))
     (stroke (width 0) (type default) (color 0 0 0 0))
   )
+  (polyline (pts (xy 46.99 109.22) (xy 46.99 111.76))
+    (stroke (width 0) (type solid) (color 0 0 0 0))
+  )
   (polyline (pts (xy 115.57 35.56) (xy 115.57 66.04))
     (stroke (width 0) (type default) (color 0 0 0 0))
   )
+  (polyline (pts (xy 48.26 109.22) (xy 49.53 109.22))
+    (stroke (width 0) (type solid) (color 0 0 0 0))
+  )
   (wire (pts (xy 191.77 71.12) (xy 193.04 71.12))
     (stroke (width 0) (type default) (color 0 0 0 0))
   )
+  (polyline (pts (xy 46.99 111.76) (xy 49.53 111.76))
+    (stroke (width 0) (type solid) (color 0 0 0 0))
+  )
   (wire (pts (xy 90.17 100.33) (xy 90.17 90.17))
     (stroke (width 0) (type default) (color 0 0 0 0))
@@
     (stroke (width 0) (type default) (color 0 0 0 0))
   )
+  (polyline (pts (xy 69.85 114.3) (xy 45.72 114.3))
+    (stroke (width 0) (type solid) (color 0 0 0 0))
+  )
   (wire (pts (xy 186.69 74.93) (xy 186.69 104.14))
     (stroke (width 0) (type default) (color 0 0 0 0))
@@
     (stroke (width 0) (type default) (color 0 0 0 0))
   )
+  (polyline (pts (xy 49.53 111.76) (xy 49.53 109.22))
+    (stroke (width 0) (type solid) (color 0 0 0 0))
+  )
   (wire (pts (xy 62.23 97.79) (xy 66.04 93.98))
     (stroke (width 0) (type default) (color 0 0 0 0))
@@
     (stroke (width 0) (type default) (color 0 0 0 0))
   )
+  (polyline (pts (xy 45.72 106.68) (xy 50.8 106.68))
+    (stroke (width 0) (type solid) (color 0 0 0 0))
+  )
   (wire (pts (xy 176.53 109.22) (xy 177.8 109.22))
     (stroke (width 0) (type default) (color 0 0 0 0))
   )
+  (polyline (pts (xy 69.85 106.68) (xy 69.85 114.3))
+    (stroke (width 0) (type solid) (color 0 0 0 0))
+  )
   (polyline (pts (xy 176.53 35.56) (xy 176.53 66.04))
     (stroke (width 0) (type default) (color 0 0 0 0))
@@
     (stroke (width 0) (type default) (color 0 0 0 0))
   )
+  (polyline (pts (xy 50.8 106.68) (xy 69.85 106.68))
+    (stroke (width 0) (type solid) (color 0 0 0 0))
+  )
   (wire (pts (xy 92.71 58.42) (xy 92.71 55.88))
     (stroke (width 0) (type default) (color 0 0 0 0))
@@
     (stroke (width 0) (type default) (color 0 0 0 0))
   )
+  (polyline (pts (xy 45.72 114.3) (xy 45.72 106.68))
+    (stroke (width 0) (type solid) (color 0 0 0 0))
+  )
   (wire (pts (xy 184.15 96.52) (xy 193.04 96.52))
     (stroke (width 0) (type default) (color 0 0 0 0))
@@
     (stroke (width 0) (type default) (color 0 0 0 0))
   )
+  (text "力" (at 69.85 116.84 0)
+    (effects (font (size 1.27 1.27)) (justify left bottom))
+  )
+  (text "minus" (at 90.17 95.25 0)
+    (effects (font (size 1.27 1.27)) (justify left bottom))
+  )
+  (text "↓" (at 68.58 118.11 0)
+    (effects (font (size 1.27 1.27)) (justify left bottom))
+  )
+  (text "↓" (at 68.58 116.84 0)
+    (effects (font (size 1.27 1.27)) (justify left bottom))
+  )
+  (text "減る" (at 53.34 116.84 0)
+    (effects (font (size 1.27 1.27)) (justify left bottom))
+  )
   (text "SWITCH" (at 116.84 38.1 0)
     (effects (font (size 1.27 1.27)) (justify left bottom))
   )
+  (text "3" (at 64.77 113.03 0)
+    (effects (font (size 1.27 1.27)) (justify left bottom))
+  )
+  (text "減る" (at 64.77 116.84 0)
+    (effects (font (size 1.27 1.27)) (justify left bottom))
+  )
+  (text "plus" (at 90.17 81.28 0)
+    (effects (font (size 1.27 1.27)) (justify left bottom))
+  )
+  (text "2" (at 53.34 113.03 0)
+    (effects (font (size 1.27 1.27)) (justify left bottom))
+  )
+  (text "4" (at 64.77 109.22 0)
+    (effects (font (size 1.27 1.27)) (justify left bottom))
+  )
+  (text "増える" (at 53.34 106.68 0)
+    (effects (font (size 1.27 1.27)) (justify left bottom))
+  )
+  (text "軸" (at 46.99 111.76 0)
+    (effects (font (size 1.27 1.27)) (justify left bottom))
+  )
   (text "DCDC" (at 34.29 41.91 0)
+    (effects (font (size 1.27 1.27)) (justify left bottom))
+  )
+  (text "増える" (at 64.77 106.68 0)
+    (effects (font (size 1.27 1.27)) (justify left bottom))
+  )
+  (text "2" (at 66.04 83.82 0)
+    (effects (font (size 1.27 1.27)) (justify left bottom))
+  )
+  (text "クランク" (at 45.72 106.68 0)
+    (effects (font (size 1.27 1.27)) (justify left bottom))
+  )
+  (text "4" (at 66.04 92.71 0)
+    (effects (font (size 1.27 1.27)) (justify left bottom))
+  )
+  (text "1" (at 57.15 83.82 0)
+    (effects (font (size 1.27 1.27)) (justify left bottom))
+  )
+  (text "1" (at 53.34 109.22 0)
+    (effects (font (size 1.27 1.27)) (justify left bottom))
+  )
+  (text "CutOff=149Hz" (at 102.87 85.09 0)
+    (effects (font (size 1.27 1.27)) (justify left bottom))
+  )
+  (text "3" (at 57.15 92.71 0)
+    (effects (font (size 1.27 1.27)) (justify left bottom))
+  )
+  (text "↓" (at 68.58 115.57 0)
     (effects (font (size 1.27 1.27)) (justify left bottom))
   )
@@
   (symbol (lib_id "Device:C_Small") (at 62.23 87.63 90) (unit 1)
     (in_bom yes) (on_board yes)
-    (property "Reference" "C2" (id 0) (at 60.96 90.17 90)
-      (effects (font (size 1.27 1.27)) (justify left))
-    )
-    (property "Value" "0.47μ" (id 1) (at 67.31 90.17 90)
+    (property "Reference" "C2" (id 0) (at 60.96 86.36 90)
+      (effects (font (size 1.27 1.27)) (justify left))
+    )
+    (property "Value" "0.47μ" (id 1) (at 68.58 86.36 90)
       (effects (font (size 1.27 1.27)) (justify left))
     )
@@
   (symbol (lib_id "Device:C_Small") (at 102.87 95.25 0) (unit 1)
     (in_bom yes) (on_board yes)
-    (property "Reference" "C7" (id 0) (at 97.79 95.25 0)
-      (effects (font (size 1.27 1.27)) (justify left))
-    )
-    (property "Value" "C_Small" (id 1) (at 92.71 97.79 0)
+    (property "Reference" "C7" (id 0) (at 105.41 96.52 0)
+      (effects (font (size 1.27 1.27)) (justify left))
+    )
+    (property "Value" "0.01u" (id 1) (at 102.87 93.98 0)
       (effects (font (size 1.27 1.27)) (justify left))
     )
@@
   (symbol (lib_id "Device:C_Small") (at 102.87 87.63 0) (unit 1)
     (in_bom yes) (on_board yes) (fields_autoplaced)
-    (property "Reference" "C6" (id 0) (at 105.1941 86.8016 0)
-      (effects (font (size 1.27 1.27)) (justify left))
-    )
-    (property "Value" "C_Small" (id 1) (at 105.1941 89.3385 0)
+    (property "Reference" "C6" (id 0) (at 105.41 86.3662 0)
+      (effects (font (size 1.27 1.27)) (justify left))
+    )
+    (property "Value" "0.1u" (id 1) (at 105.41 88.9062 0)
       (effects (font (size 1.27 1.27)) (justify left))
     )
@@
   (symbol (lib_id "Device:R_Small") (at 97.79 85.09 90) (unit 1)
     (in_bom yes) (on_board yes)
-    (property "Reference" "R1" (id 0) (at 92.71 82.55 90))
-    (property "Value" "R_Small" (id 1) (at 97.79 82.55 90))
+    (property "Reference" "R1" (id 0) (at 97.79 85.09 90))
+    (property "Value" "5.1k" (id 1) (at 93.98 83.82 90))
     (property "Footprint" "Resistor_SMD:R_0603_1608Metric_Pad0.98x0.95mm_HandSolder" (id 2) (at 97.79 85.09 0)
       (effects (font (size 1.27 1.27)) hide)
@@
   (symbol (lib_id "Device:C_Small") (at 102.87 80.01 0) (unit 1)
     (in_bom yes) (on_board yes)
-    (property "Reference" "C5" (id 0) (at 97.79 77.47 0)
-      (effects (font (size 1.27 1.27)) (justify left))
-    )
-    (property "Value" "C_Small" (id 1) (at 92.71 80.01 0)
+    (property "Reference" "C5" (id 0) (at 105.41 78.74 0)
+      (effects (font (size 1.27 1.27)) (justify left))
+    )
+    (property "Value" "0.01u" (id 1) (at 102.87 81.28 0)
       (effects (font (size 1.27 1.27)) (justify left))
     )
@@
   (symbol (lib_id "Device:R_Small") (at 97.79 90.17 90) (unit 1)
     (in_bom yes) (on_board yes)
-    (property "Reference" "R2" (id 0) (at 92.71 92.71 90))
-    (property "Value" "R_Small" (id 1) (at 97.79 92.71 90))
+    (property "Reference" "R2" (id 0) (at 97.79 90.17 90))
+    (property "Value" "5.1k" (id 1) (at 93.98 88.9 90))
     (property "Footprint" "Resistor_SMD:R_0603_1608Metric_Pad0.98x0.95mm_HandSolder" (id 2) (at 97.79 90.17 0)
       (effects (font (size 1.27 1.27)) hide)
@@
     )
     (path "/df747819-65e1-4418-8b66-3be87a1662ea"
-      (reference "C5") (unit 1) (value "C_Small") (footprint "Capacitor_SMD:C_0603_1608Metric_Pad1.08x0.95mm_HandSolder")
+      (reference "C5") (unit 1) (value "0.01u") (footprint "Capacitor_SMD:C_0603_1608Metric_Pad1.08x0.95mm_HandSolder")
     )
     (path "/9574c506-77a6-484b-a3ed-87b28c19542e"
-      (reference "C6") (unit 1) (value "C_Small") (footprint "Capacitor_SMD:C_0603_1608Metric_Pad1.08x0.95mm_HandSolder")
+      (reference "C6") (unit 1) (value "0.1u") (footprint "Capacitor_SMD:C_0603_1608Metric_Pad1.08x0.95mm_HandSolder")
     )
     (path "/8eef5ee4-ce00-4f9e-96ed-0a8313f76431"
-      (reference "C7") (unit 1) (value "C_Small") (footprint "Capacitor_SMD:C_0603_1608Metric_Pad1.08x0.95mm_HandSolder")
+      (reference "C7") (unit 1) (value "0.01u") (footprint "Capacitor_SMD:C_0603_1608Metric_Pad1.08x0.95mm_HandSolder")
     )
     (path "/ee49c403-5615-4006-b408-b9d33c48488d"
@@
     )
     (path "/d560799b-91f1-4f47-a403-0be848989901"
-      (reference "R1") (unit 1) (value "R_Small") (footprint "Resistor_SMD:R_0603_1608Metric_Pad0.98x0.95mm_HandSolder")
+      (reference "R1") (unit 1) (value "5.1k") (footprint "Resistor_SMD:R_0603_1608Metric_Pad0.98x0.95mm_HandSolder")
     )
     (path "/ebad1c30-f3aa-4bb7-835c-16197b5f9a6d"
-      (reference "R2") (unit 1) (value "R_Small") (footprint "Resistor_SMD:R_0603_1608Metric_Pad0.98x0.95mm_HandSolder")
+      (reference "R2") (unit 1) (value "5.1k") (footprint "Resistor_SMD:R_0603_1608Metric_Pad0.98x0.95mm_HandSolder")
     )
     (path "/84934404-283e-4110-ad68-d793fbe50bd6"
